File: Hardware/monkey_arduino_shield/monkey_arduino_shield.kicad_pcb (KiCad board)
At the start: 2 copper layers, 68.6 x 53.3 mm, 28 parts, among them J1 Speaker_OUT, J2 Barrel_Jack, J3 Screw_Terminal_01x03, J4 Screw_Terminal_01x03, J5 MIC_IN, P1 Power, P2 Analog, P3 Digital, P4 Digital, P5 CONN_01X01, P6 CONN_01X01, P7 CONN_01X01, P8 CONN_01X01, U1 W25Q128JVS, U2 SN74LVC2T45DCUR, U3 SN74LVC2T45DCUR, U4 TPA2005D1DRB, U5 AMS1117-5.0

Commit message: Hardware Revision in Progress
Parts:
- moved F1 75.4 mm to (133.9, 88.3), turned to 270 degrees
- moved FB1 68.0 mm to (128.8, 88.3), turned to 270 degrees
- moved C3 60.7 mm to (135.1, 92.1)
- moved C4 60.5 mm to (135.1, 95.9)
- moved U5 60.4 mm to (158.0, 95.9)
- moved J2 54.6 mm to (119.9, 87.0), turned to 0 degrees
- moved J5 50.3 mm to (164.3, 116.2)
- moved J4 43.6 mm to (212.6, 70.5)
- moved J3 39.8 mm to (198.6, 70.5)
- moved J1 32.1 mm to (147.8, 113.7)
- moved U1 31.9 mm to (160.5, 85.7)
- moved D1 6.84 mm to (125.0, 88.3)
Connections:
- J3 pad 3: +5V -> /Vin
- J4 pad 3: +5V -> /Vin
Routing:
- net GND: track 169.3 -> 0.00 mm, vias 3 -> 0
- net +5V: track 118.4 -> 0.00 mm, vias 2 -> 0
- net +3V3: track 95.9 -> 0.00 mm, vias 3 -> 0
- net /A0: track 60.2 -> 0.00 mm
- net /LV_MOSI: track 36.1 -> 0.00 mm, vias 2 -> 0
- net /6(**): track 32.5 -> 0.00 mm
- net /LV_SCK: track 30.4 -> 0.00 mm
- net /A1: track 29.1 -> 0.00 mm, vias 3 -> 0
- net /13(HV_SCK): track 22.6 -> 0.00 mm
- net /11(HV_MOSI): track 18.9 -> 0.00 mm, vias 2 -> 0
- net /5(**): track 14.1 -> 0.00 mm
- net /12(HV_MISO): track 10.1 -> 0.00 mm, vias 2 -> 0
- net /LV_MISO: track 9.82 -> 0.00 mm
- net Net-(J1-Pad1): track 6.27 -> 0.00 mm
- net Net-(R2-Pad1): track 6.14 -> 0.00 mm
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- removed copper zone on B.Cu, net GND

Commit message: Final PCB Revision
Parts:
- removed C1, C2: 1u, Capacitor_SMD:C_1206_3216Metric
- removed R1: 10K, Resistor_SMD:R_0603_1608Metric
- removed R2, R3: 150k, Resistor_SMD:R_0603_1608Metric
- removed U2, U3: SN74LVC2T45DCUR, Package_SO:VSSOP-8_2.4x2.1mm_P0.5mm
- removed U4: TPA2005D1DRB, Package_SO:MSOP-8-1EP_3x3mm_P0.65mm_EP1.68x1.88mm
- added J10: IO_Switch_3, Connector_PinSocket_2.54mm:PinSocket_1x02_P2.54mm_Vertical, F.Cu at (166.9, 84.5)
- added J11: IO_Switch_4, Connector_PinSocket_2.54mm:PinSocket_1x02_P2.54mm_Vertical, F.Cu at (163.1, 84.5)
- added J6: POT_IN, Connector_PinSocket_2.54mm:PinSocket_1x03_P2.54mm_Vertical, F.Cu at (113.5, 88.3)
- added J7: Power_Switch, Connector_PinSocket_2.54mm:PinSocket_1x02_P2.54mm_Vertical, F.Cu at (113.5, 118.7)
- added J8: IO_Switch_1, Connector_PinSocket_2.54mm:PinSocket_1x02_P2.54mm_Vertical, F.Cu at (174.5, 84.5)
- added J9: IO_Switch_2, Connector_PinSocket_2.54mm:PinSocket_1x02_P2.54mm_Vertical, F.Cu at (170.7, 84.5)
- C3, C4: footprint Capacitor_SMD:C_1206_3216Metric -> Capacitor_THT:CP_Radial_D5.0mm_P2.00mm
- D1: footprint Diode_SMD:D_0603_1608Metric -> Diode_THT:D_DO-41_SOD81_P7.62mm_Horizontal
- F1: value 500mA -> 1A; footprint Fuse:Fuse_0603_1608Metric -> Fuse:Fuseholder_Blade_Mini_Keystone_3568
- FB1: footprint Inductor_SMD:L_0201_0603Metric -> Diode_THT:D_DO-41_SOD81_P7.62mm_Horizontal
- J1: footprint TerminalBlock:TerminalBlock_bornier-2_P5.08mm -> Connector_PinSocket_2.54mm:PinSocket_1x02_P2.54mm_Vertical
- J2: footprint Connector_BarrelJack:BarrelJack_Horizontal -> Socket_Arduino_Uno:BarrelJack_Horizontal_Helmer_Version
- J3: value Screw_Terminal_01x03 -> MOTOR_1; footprint TerminalBlock:TerminalBlock_bornier-3_P5.08mm -> Connector_PinSocket_2.54mm:PinSocket_1x03_P2.54mm_Vertical
- J4: value Screw_Terminal_01x03 -> MOTOR_2; footprint TerminalBlock:TerminalBlock_bornier-3_P5.08mm -> Connector_PinSocket_2.54mm:PinSocket_1x03_P2.54mm_Vertical
- J5: footprint TerminalBlock:TerminalBlock_bornier-3_P5.08mm -> Connector_PinSocket_2.54mm:PinSocket_1x03_P2.54mm_Vertical
- U1: value W25Q128JVS -> TPA2005D1-Breakout; footprint Package_SO:SOIC-8_5.23x5.23mm_P1.27mm -> Socket_Arduino_Uno:TDA_Breakout_Board
- moved J4 55.8 mm to (158.0, 81.9), turned to 0 degrees
- moved J3 45.9 mm to (154.2, 81.9), turned to 0 degrees
- moved J1 33.6 mm to (177.0, 97.2), turned to 0 degrees
- moved D1 31.1 mm to (131.3, 118.7), turned to 180 degrees
- moved U1 29.6 mm to (131.3, 80.6)
- moved C4 26.7 mm to (159.3, 107.3)
- moved FB1 24.3 mm to (131.3, 112.4), turned to 180 degrees
- moved C3 22.5 mm to (151.6, 107.3)
- moved U5 20.4 mm to (156.7, 116.2)
- moved J2 20.3 mm to (119.9, 107.3)
- moved F1 17.0 mm to (126.2, 103.5), turned to 0 degrees
- moved J5 15.5 mm to (177.0, 107.3), turned to 0 degrees
Connections:
- J1 pad 1: Net-(J1-Pad1) -> GND
- J1 pad 2: GND -> Net-(J1-Pad2)
- J2 pad 1: Net-(D1-Pad2) -> Net-(J2-Pad1)
- P1 pad 1: Net-(P1-Pad1) -> (no net)
- P1 pad 2: /IOREF -> (no net)
- P1 pad 3: /Reset -> (no net)
- P2 pad 3: /A2 -> (no net)
- P2 pad 4: /A3 -> (no net)
- P2 pad 5: /A4(SDA) -> (no net)
- P2 pad 6: /A5(SCL) -> (no net)
- P3 pad 1: /A5(SCL_) -> (no net)
- P3 pad 10: /8 -> (no net)
- P3 pad 2: /A4(SDA_) -> (no net)
- P3 pad 3: /AREF -> (no net)
- P3 pad 5: /13(HV_SCK) -> (no net)
- P3 pad 6: /12(HV_MISO) -> (no net)
- P3 pad 7: /11(HV_MOSI) -> (no net)
- P3 pad 8: /10(**/SS) -> (no net)
- P3 pad 9: /9(**) -> (no net)
- P4 pad 1: /7 -> (no net)
- P4 pad 4: /4 -> (no net)
- P5 pad 1: Net-(P5-Pad1) -> (no net)
- P6 pad 1: Net-(P6-Pad1) -> (no net)
- P7 pad 1: Net-(P7-Pad1) -> (no net)
- P8 pad 1: Net-(P8-Pad1) -> (no net)
- U1 pad 1: +3V3 -> Net-(J1-Pad2)
- U1 pad 2: /LV_MISO -> GND
- U1 pad 3: Net-(U1-Pad3) -> GND
- U1 pad 4: GND -> +5V
- U1 pad 5: /LV_MOSI -> (no net)
- U1 pad 6: /LV_SCK -> /A1
- U1 pad 7: Net-(U1-Pad7) -> GND
- U1 pad 8: +3V3 -> Net-(J6-Pad1)
Routing:
- net /A1: track 0.00 -> 53.2 mm
- net /Vin: track 0.00 -> 42.2 mm
- net +5V: track 0.00 -> 41.8 mm, vias 0 -> 2
- net +3V3: track 0.00 -> 40.3 mm, vias 0 -> 1
- net Net-(J1-Pad2): track 0.00 -> 37.4 mm
- net Net-(C3-Pad1): track 0.00 -> 25.9 mm
- net /A0: track 0.00 -> 22.2 mm
- net GND: track 0.00 -> 21.9 mm
- net /6(**): track 0.00 -> 14.1 mm
- net Net-(J2-Pad1): track 0.00 -> 13.3 mm
- net Net-(F1-Pad1): track 0.00 -> 11.7 mm
- net /5(**): track 0.00 -> 11.2 mm
- net /3(**): track 0.00 -> 10.5 mm
- net Net-(D1-Pad1): track 0.00 -> 10.3 mm
- net Net-(D1-Pad2): track 0.00 -> 10.2 mm
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- added copper zone on B.Cu, net GND
Other:
- outline, holes or cut-outs redrawn
- rule via_min_size: 0.4 -> 0.4572
- board text added: "Andrew, Helmut, Jennifer, and Tyler"
- board text added: "ECE3872 - Section C, Group 2"
