File: Hardware/monkey_arduino_shield/monkey_arduino_shield.sch (KiCad schematic (older format))
At the start: 28 parts, among them J1 Speaker_OUT, J2 Barrel_Jack, J3 Screw_Terminal_01x03, J4 Screw_Terminal_01x03, J5 MIC_IN, P1 Power, P2 Analog, P3 Digital, P4 Digital, P5 CONN_01X01, P6 CONN_01X01, P7 CONN_01X01, P8 CONN_01X01, U1 W25Q128JVS, U2 SN74LVC2T45DCUR, U3 SN74LVC2T45DCUR, U4 TPA2005D1DRB, U5 AMS1117-5.0

Commit message: Modified power for motors.
Other:
- note added: "POWER SUPPLY"
- moved on the sheet: C3, C4, D1, F1, FB1, J2, U5
Changed lines of the file:
@@
-$EndComp
-$Comp
-L power:+5V #PWR0114
-U 1 1 61685866
-P 2700 3000
-F 0 "#PWR0114" H 2700 2850 50  0001 C CNN
-F 1 "+5V" H 2500 3050 50  0000 C CNN
-F 2 "" H 2700 3000 50  0001 C CNN
-F 3 "" H 2700 3000 50  0001 C CNN
-	1    2700 3000
-	1    0    0    -1
-$EndComp
-$Comp
-L power:+5V #PWR0115
-U 1 1 61685A9C
-P 2700 2450
-F 0 "#PWR0115" H 2700 2300 50  0001 C CNN
-F 1 "+5V" H 2500 2500 50  0000 C CNN
-F 2 "" H 2700 2450 50  0001 C CNN
-F 3 "" H 2700 2450 50  0001 C CNN
-	1    2700 2450
-	1    0    0    -1
 $EndComp
 $Comp
@@
 Wire Wire Line
 	4300 3050 4300 3000
+Text Label 2700 2450 0    50   ~ 0
+Vin
+Text Label 2700 3000 0    50   ~ 0
+Vin
 $Comp
 L Connector:Barrel_Jack J2
 U 1 1 614A55C8
-P 800 4400
-F 0 "J2" H 857 4725 50  0000 C CNN
-F 1 "Barrel_Jack" H 857 4634 50  0000 C CNN
-F 2 "Connector_BarrelJack:BarrelJack_Horizontal" H 850 4360 50  0001 C CNN
-F 3 "~" H 850 4360 50  0001 C CNN
-	1    800  4400
+P 4450 4500
+F 0 "J2" H 4507 4825 50  0000 C CNN
+F 1 "Barrel_Jack" H 4507 4734 50  0000 C CNN
+F 2 "Connector_BarrelJack:BarrelJack_Horizontal" H 4500 4460 50  0001 C CNN
+F 3 "~" H 4500 4460 50  0001 C CNN
+	1    4450 4500
 	1    0    0    -1
 $EndComp
@@
 L Diode:1N4001 D1
 U 1 1 614A714C
-P 1350 4300
-F 0 "D1" H 1350 4083 50  0000 C CNN
-F 1 "B5819W" H 1350 4174 50  0000 C CNN
-F 2 "Diode_SMD:D_0603_1608Metric" H 1350 4125 50  0001 C CNN
-F 3 "http://www.vishay.com/docs/88503/1n4001.pdf" H 1350 4300 50  0001 C CNN
-	1    1350 4300
+P 5000 4400
+F 0 "D1" H 5000 4183 50  0000 C CNN
+F 1 "B5819W" H 5000 4274 50  0000 C CNN
+F 2 "Diode_SMD:D_0603_1608Metric" H 5000 4225 50  0001 C CNN
+F 3 "http://www.vishay.com/docs/88503/1n4001.pdf" H 5000 4400 50  0001 C CNN
+	1    5000 4400
 	-1   0    0    1
 $EndComp
@@
 L Device:Ferrite_Bead_Small FB1
 U 1 1 614A8763
-P 1900 4300
-F 0 "FB1" V 1663 4300 50  0000 C CNN
-F 1 "100 Ohm @ 100 MHz" V 1754 4300 50  0000 C CNN
-F 2 "Inductor_SMD:L_0201_0603Metric" V 1830 4300 50  0001 C CNN
-F 3 "~" H 1900 4300 50  0001 C CNN
-	1    1900 4300
+P 5550 4400
+F 0 "FB1" V 5313 4400 50  0000 C CNN
+F 1 "100 Ohm @ 100 MHz" V 5404 4400 50  0000 C CNN
+F 2 "Inductor_SMD:L_0201_0603Metric" V 5480 4400 50  0001 C CNN
+F 3 "~" H 5550 4400 50  0001 C CNN
+	1    5550 4400
 	0    1    1    0
 $EndComp
@@
 L Device:Fuse_Small F1
 U 1 1 614A952C
-P 2350 4300
-F 0 "F1" H 2350 4485 50  0000 C CNN
-F 1 "500mA" H 2350 4394 50  0000 C CNN
-F 2 "Fuse:Fuse_0603_1608Metric" H 2350 4300 50  0001 C CNN
-F 3 "~" H 2350 4300 50  0001 C CNN
-	1    2350 4300
+P 6000 4400
+F 0 "F1" H 6000 4585 50  0000 C CNN
+F 1 "500mA" H 6000 4494 50  0000 C CNN
+F 2 "Fuse:Fuse_0603_1608Metric" H 6000 4400 50  0001 C CNN
+F 3 "~" H 6000 4400 50  0001 C CNN
+	1    6000 4400
 	1    0    0    -1
 $EndComp
@@
 L Regulator_Linear:AMS1117-5.0 U5
 U 1 1 614AA01B
-P 2950 4300
-F 0 "U5" H 2950 4542 50  0000 C CNN
-F 1 "AMS1117-5.0" H 2950 4451 50  0000 C CNN
-F 2 "Package_TO_SOT_SMD:SOT-223-3_TabPin2" H 2950 4500 50  0001 C CNN
-F 3 "http://www.advanced-monolithic.com/pdf/ds1117.pdf" H 3050 4050 50  0001 C CNN
-	1    2950 4300
-	1    0    0    -1
-$EndComp
-Wire Wire Line
-	1100 4300 1200 4300
-Wire Wire Line
-	1500 4300 1800 4300
-Wire Wire Line
-	2000 4300 2250 4300
-Wire Wire Line
-	2450 4300 2550 4300
+P 6600 4400
+F 0 "U5" H 6600 4642 50  0000 C CNN
+F 1 "AMS1117-5.0" H 6600 4551 50  0000 C CNN
+F 2 "Package_TO_SOT_SMD:SOT-223-3_TabPin2" H 6600 4600 50  0001 C CNN
+F 3 "http://www.advanced-monolithic.com/pdf/ds1117.pdf" H 6700 4150 50  0001 C CNN
+	1    6600 4400
+	1    0    0    -1
+$EndComp
+Wire Wire Line
+	4750 4400 4850 4400
+Wire Wire Line
+	5150 4400 5450 4400
+Wire Wire Line
+	5650 4400 5900 4400
+Wire Wire Line
+	6100 4400 6200 4400
 $Comp
 L Device:CP_Small C3
 U 1 1 614C7832
-P 2550 4400
-F 0 "C3" H 2638 4446 50  0000 L CNN
-F 1 "10u" H 2638 4355 50  0000 L CNN
-F 2 "Capacitor_SMD:C_1206_3216Metric" H 2550 4400 50  0001 C CNN
-F 3 "~" H 2550 4400 50  0001 C CNN
-	1    2550 4400
-	1    0    0    -1
-$EndComp
-Connection ~ 2550 4300
-Wire Wire Line
-	2550 4300 2650 4300
+P 6200 4500
+F 0 "C3" H 6288 4546 50  0000 L CNN
+F 1 "10u" H 6288 4455 50  0000 L CNN
+F 2 "Capacitor_SMD:C_1206_3216Metric" H 6200 4500 50  0001 C CNN
+F 3 "~" H 6200 4500 50  0001 C CNN
+	1    6200 4500
+	1    0    0    -1
+$EndComp
+Connection ~ 6200 4400
+Wire Wire Line
+	6200 4400 6300 4400
 $Comp
 L Device:CP_Small C4
 U 1 1 614C8737
-P 3400 4400
-F 0 "C4" H 3488 4446 50  0000 L CNN
-F 1 "10u" H 3488 4355 50  0000 L CNN
-F 2 "Capacitor_SMD:C_1206_3216Metric" H 3400 4400 50  0001 C CNN
-F 3 "~" H 3400 4400 50  0001 C CNN
-	1    3400 4400
-	1    0    0    -1
-$EndComp
-Wire Wire Line
-	3250 4300 3400 4300
-Wire Wire Line
-	2950 4600 3400 4600
-Wire Wire Line
-	3400 4600 3400 4500
-Wire Wire Line
-	2950 4600 2550 4600
-Wire Wire Line
-	2550 4600 2550 4500
-Connection ~ 2950 4600
+P 7050 4500
+F 0 "C4" H 7138 4546 50  0000 L CNN
+F 1 "10u" H 7138 4455 50  0000 L CNN
+F 2 "Capacitor_SMD:C_1206_3216Metric" H 7050 4500 50  0001 C CNN
+F 3 "~" H 7050 4500 50  0001 C CNN
+	1    7050 4500
+	1    0    0    -1
+$EndComp
+Wire Wire Line
+	6900 4400 7050 4400
+Wire Wire Line
+	6600 4700 7050 4700
+Wire Wire Line
+	7050 4700 7050 4600
+Wire Wire Line
+	6600 4700 6200 4700
+Wire Wire Line
+	6200 4700 6200 4600
+Connection ~ 6600 4700
 $Comp
 L power:GND #PWR0124
 U 1 1 614D1996
-P 2950 4600
-F 0 "#PWR0124" H 2950 4350 50  0001 C CNN
-F 1 "GND" H 2955 4427 50  0000 C CNN
-F 2 "" H 2950 4600 50  0001 C CNN
-F 3 "" H 2950 4600 50  0001 C CNN
-	1    2950 4600
+P 6600 4700
+F 0 "#PWR0124" H 6600 4450 50  0001 C CNN
+F 1 "GND" H 6605 4527 50  0000 C CNN
+F 2 "" H 6600 4700 50  0001 C CNN
+F 3 "" H 6600 4700 50  0001 C CNN
+	1    6600 4700
 	1    0    0    -1
 $EndComp
@@
 L power:GND #PWR0125
 U 1 1 614D1D87
-P 1100 4500
-F 0 "#PWR0125" H 1100 4250 50  0001 C CNN
-F 1 "GND" H 1105 4327 50  0000 C CNN
-F 2 "" H 1100 4500 50  0001 C CNN
-F 3 "" H 1100 4500 50  0001 C CNN
-	1    1100 4500
-	1    0    0    -1
-$EndComp
-Text Label 3400 4300 0    50   ~ 0
+P 4750 4600
+F 0 "#PWR0125" H 4750 4350 50  0001 C CNN
+F 1 "GND" H 4755 4427 50  0000 C CNN
+F 2 "" H 4750 4600 50  0001 C CNN
+F 3 "" H 4750 4600 50  0001 C CNN
+	1    4750 4600
+	1    0    0    -1
+$EndComp
+Text Label 7050 4400 0    50   ~ 0
 Vin
+Wire Notes Line style solid
+	7400 4050 4150 4050
+Wire Notes Line style solid
+	4150 4050 4150 5350
+Wire Notes Line style solid
+	4150 5350 7400 5350
+Wire Notes Line style solid
+	7400 5350 7400 4050
+Text Notes 4200 5300 0    50   ~ 0
+POWER SUPPLY
 $EndSCHEMATC

Commit message: Final PCB Revision
Parts:
- removed C1, C2: 1u, Capacitor_SMD:C_1206_3216Metric, symbol Device:C_Small
- removed R1: 10K, Resistor_SMD:R_0603_1608Metric, symbol Device:R_Small
- removed R2, R3: 150k, Resistor_SMD:R_0603_1608Metric, symbol Device:R_Small
- removed U1: W25Q128JVS, Package_SO:SOIC-8_5.23x5.23mm_P1.27mm, symbol Memory_Flash:W25Q128JVS
- removed U2, U3: SN74LVC2T45DCUR, Package_SO:VSSOP-8_2.4x2.1mm_P0.5mm, symbol Logic_LevelTranslator:SN74LVC2T45DCUR
- removed U4: TPA2005D1DRB, Package_SO:MSOP-8-1EP_3x3mm_P0.65mm_EP1.68x1.88mm, symbol monkey_arduino_shield-rescue:TPA2005D1DRB-SparkFun-AnalogIC
- added J10: IO_Switch_3, Connector_PinSocket_2.54mm:PinSocket_1x02_P2.54mm_Vertical, symbol Connector:Screw_Terminal_01x02
- added J11: IO_Switch_4, Connector_PinSocket_2.54mm:PinSocket_1x02_P2.54mm_Vertical, symbol Connector:Screw_Terminal_01x02
- added J6: POT_IN, Connector_PinSocket_2.54mm:PinSocket_1x03_P2.54mm_Vertical, symbol Connector:Screw_Terminal_01x03
- added J7: Power_Switch, Connector_PinSocket_2.54mm:PinSocket_1x02_P2.54mm_Vertical, symbol Connector:Screw_Terminal_01x02
- added J8: IO_Switch_1, Connector_PinSocket_2.54mm:PinSocket_1x02_P2.54mm_Vertical, symbol Connector:Screw_Terminal_01x02
- added J9: IO_Switch_2, Connector_PinSocket_2.54mm:PinSocket_1x02_P2.54mm_Vertical, symbol Connector:Screw_Terminal_01x02
- added U1: TPA2005D1-Breakout, Socket_Arduino_Uno:TDA_Breakout_Board, symbol tpa2005d1-breakout:TPA2005D1-Breakout
- C3, C4: footprint Capacitor_SMD:C_1206_3216Metric -> Capacitor_THT:CP_Radial_D5.0mm_P2.00mm
- D1: footprint Diode_SMD:D_0603_1608Metric -> Diode_THT:D_DO-41_SOD81_P7.62mm_Horizontal
- F1: value 500mA -> 1A; footprint Fuse:Fuse_0603_1608Metric -> Fuse:Fuseholder_Blade_Mini_Keystone_3568
- FB1: footprint Inductor_SMD:L_0201_0603Metric -> Diode_THT:D_DO-41_SOD81_P7.62mm_Horizontal
- J1: footprint TerminalBlock:TerminalBlock_bornier-2_P5.08mm -> Connector_PinSocket_2.54mm:PinSocket_1x02_P2.54mm_Vertical
- J3: value Screw_Terminal_01x03 -> MOTOR_1; footprint TerminalBlock:TerminalBlock_bornier-3_P5.08mm -> Connector_PinSocket_2.54mm:PinSocket_1x03_P2.54mm_Vertical
- J4: value Screw_Terminal_01x03 -> MOTOR_2; footprint TerminalBlock:TerminalBlock_bornier-3_P5.08mm -> Connector_PinSocket_2.54mm:PinSocket_1x03_P2.54mm_Vertical
- J5: footprint TerminalBlock:TerminalBlock_bornier-3_P5.08mm -> Connector_PinSocket_2.54mm:PinSocket_1x03_P2.54mm_Vertical
Connections:
- net labels removed: LV_MISO, LV_MOSI, LV_SCK
- no-connect marks 9 -> 6
Other:
- note added: "DIGITAL INPUTS"
- note added: "MICROPHONE INPUT (PREAMPLIFIED), AUDIO OUTPUT"
- note removed: "MICROPHONE INPUT (PREAMPLIFIED)"
- note removed: "SPI LEVEL SHIFT (5V -> 3.3V)"
- note removed: "SRAM EXPANSION"
- moved on the sheet: C3, C4, D1, F1, FB1, J1, J2, J3, J4, J5, U5

Commit message: Updated Barrel Jack
Parts:
- J2: footprint Connector_BarrelJack:BarrelJack_Horizontal -> Socket_Arduino_Uno:BarrelJack_Horizontal_Helmer_Version
Changed lines of the file:
@@
 F 0 "J2" H 2557 3175 50  0000 C CNN
 F 1 "Barrel_Jack" H 2557 3084 50  0000 C CNN
-F 2 "Connector_BarrelJack:BarrelJack_Horizontal" H 2550 2810 50  0001 C CNN
+F 2 "Socket_Arduino_Uno:BarrelJack_Horizontal_Helmer_Version" H 2550 2810 50  0001 C CNN
 F 3 "~" H 2550 2810 50  0001 C CNN
 	1    2500 2850
